Commit message: Change robot description: remove hands, replace with box for self-filtering

File: husky_description/urdf/dual_arm_husky.urdf.xacro (robot description, xacro)
@@ -1211,5 +1211,5 @@
   </link>
   <!-- virtual measurement frame -->
-  <joint name="l_robotiq_fts300_measurment_joint" type="fixed">
+  <joint name="l_robotiq_fts300_measurement_joint" type="fixed">
     <origin rpy="0 0 0" xyz="0 0 0.01625"/>
     <parent link="l_robotiq_fts300_fts_robotside"/>
@@ -1252,5 +1252,5 @@
   </link>
   <!-- virtual measurement frame -->
-  <joint name="r_robotiq_fts300_measurment_joint" type="fixed">
+  <joint name="r_robotiq_fts300_measurement_joint" type="fixed">
     <origin rpy="0 0 0" xyz="0 0 0.01625"/>
     <parent link="r_robotiq_fts300_fts_robotside"/>
@@ -1272,11 +1272,9 @@
   </joint>
   <!-- Insert the fingers -->
-  <!-- Link list -->
-  <!-- Link 0 -->
-  <link name="l_finger_1_link_0">
-    <visual>
-      <origin rpy="0 0 0" xyz="0 0 0"/>
-      <geometry>
-        <mesh filename="package://robotiq_s_model_visualization/meshes/s-model_articulated/visual/link_0.STL"/>
+  <!-- Link palm -->
+  <link name="l_palm">
+    <visual>
+      <geometry>
+        <mesh filename="package://robotiq_s_model_visualization/meshes/s-model_articulated/visual/palm.STL"/>
       </geometry>
       <material name="green">
@@ -1284,1697 +1282,9 @@
       </material>
     </visual>
-    <collision>
-      <origin rpy="0 0 0" xyz="0 0 0"/>
-      <geometry>
-        <mesh filename="package://robotiq_s_model_visualization/meshes/s-model_articulated/collision/link_0.STL"/>
-      </geometry>
-      <material name="yellow">
-        <color rgba="0 1 1 1"/>
-      </material>
-    </collision>
-    <inertial>
-      <mass value="0.1"/>
-      <origin xyz="-0.01 0 0"/>
-      <inertia ixx="0.000018" ixy="0" ixz="0" iyy="0.000025" iyz="0" izz="0.000025"/>
-    </inertial>
-  </link>
-  <gazebo reference="l_finger_1_link_0">
-    <mu1>1.1</mu1>
-    <mu2>1.1</mu2>
-  </gazebo>
-  <!-- Link 1 -->
-  <link name="l_finger_1_link_1">
-    <visual>
-      <origin rpy="0 0 1.5708" xyz="0 0.05717 0"/>
-      <geometry>
-        <mesh filename="package://robotiq_s_model_visualization/meshes/s-model_articulated/visual/link_1.STL"/>
-      </geometry>
-      <material name="green"/>
-    </visual>
-    <collision>
-      <origin rpy="0 0 1.5708" xyz="0 0.05717 0"/>
-      <geometry>
-        <mesh filename="package://robotiq_s_model_visualization/meshes/s-model_articulated/collision/link_1.STL"/>
-      </geometry>
-      <material name="yellow">
-        <color rgba="0 1 1 1"/>
-      </material>
-    </collision>
-    <inertial>
-      <origin rpy="0 0 1.5708" xyz="0.00053 0.03218 0"/>
-      <mass value="0.047"/>
-      <inertia ixx="0.00000499332" ixy="0.00000091312" ixz="-0.00000000120" iyy="0.00006434531" iyz="-0.00000000007" izz="0.00006061917"/>
-    </inertial>
-  </link>
-  <gazebo reference="l_finger_1_link_1">
-    <mu1>1.1</mu1>
-    <mu2>1.1</mu2>
-  </gazebo>
-  <!-- Link 2 -->
-  <link name="l_finger_1_link_2">
-    <visual>
-      <origin rpy="0 0 1.5708" xyz="0 0.03810 0.0075"/>
-      <geometry>
-        <mesh filename="package://robotiq_s_model_visualization/meshes/s-model_articulated/visual/link_2.STL"/>
-      </geometry>
-      <material name="green"/>
-    </visual>
-    <collision>
-      <origin rpy="0 0 1.5708" xyz="0 0.03810 0.0075"/>
-      <geometry>
-        <mesh filename="package://robotiq_s_model_visualization/meshes/s-model_articulated/collision/link_2.STL"/>
-      </geometry>
-      <material name="yellow"/>
-    </collision>
-    <inertial>
-      <origin rpy="0 0 1.5708" xyz="0.00048 0.02167 0.00018"/>
-      <mass value="0.03284"/>
-      <inertia ixx="0.00000348008" ixy="0.00000031940" ixz="0.00000013041" iyy="0.00002248123" iyz="0.00000000291" izz="0.00001986346"/>
-    </inertial>
-  </link>
-  <gazebo reference="l_finger_1_link_2">
-    <mu1>1.1</mu1>
-    <mu2>1.1</mu2>
-  </gazebo>
-  <!-- Link 3 -->
-  <link name="l_finger_1_link_3">
-    <visual>
-      <origin rpy="0 0 0" xyz="0 0 0"/>
-      <geometry>
-        <mesh filename="package://robotiq_s_model_visualization/meshes/s-model_articulated/visual/link_3.STL"/>
-      </geometry>
-      <material name="green"/>
-    </visual>
-    <collision>
-      <origin rpy="0 0 0" xyz="0 0 0"/>
-      <geometry>
-        <mesh filename="package://robotiq_s_model_visualization/meshes/s-model_articulated/collision/link_3.STL"/>
-      </geometry>
-      <material name="yellow"/>
-    </collision>
-    <inertial>
-      <origin rpy="0 0 0" xyz="0.01626 0.00049 0.0002"/>
-      <mass value="0.03354"/>
-      <inertia ixx="0.00000305151" ixy="0.00000089792" ixz="0.00000000249" iyy="0.00001427978" iyz="-0.00000001191" izz="0.00001264126"/>
-    </inertial>
-  </link>
-  <gazebo reference="l_finger_1_link_3">
-    <mu1>1.1</mu1>
-    <mu2>1.1</mu2>
-  </gazebo>
-  <!-- Link proximal actuating hinge -->
-  <link name="l_finger_1_link_proximal_actuating_hinge">
-    <visual>
-      <origin rpy="0 0 0" xyz="0.01429 0 0"/>
-      <geometry>
-        <box size="0.02858 .0075 .002"/>
-      </geometry>
-    </visual>
-    <collision>
-      <origin rpy="0 0 0" xyz="0.01429 0 0"/>
-      <geometry>
-        <box size="0.02858 .0075 .002"/>
-      </geometry>
-    </collision>
-    <inertial>
-      <origin rpy="0 0 0" xyz="0.0012 -0.00162 -0.00161"/>
-      <mass value="0.02647"/>
-      <inertia ixx="0.00000156447" ixy="0.000000236226" ixz="-0.00000014862" iyy="0.00000221068" iyz="-0.00000014369" izz="0.00000323175"/>
-    </inertial>
-  </link>
-  <gazebo reference="l_finger_1_link_proximal_actuating_hinge">
-    <mu1>1.1</mu1>
-    <mu2>1.1</mu2>
-  </gazebo>
-  <!-- Link paraproximal actuating hinge -->
-  <link name="l_finger_1_link_paraproximal_actuating_hinge">
-    <visual>
-      <origin rpy="0 0 0" xyz="0.01143 0 0"/>
-      <geometry>
-        <box size="0.02286 .0075 .002"/>
-      </geometry>
-    </visual>
-    <collision>
-      <origin rpy="0 0 0" xyz="0.01143 0 0"/>
-      <geometry>
-        <box size="0.02286 .0075 .002"/>
-      </geometry>
-    </collision>
-    <inertial>
-      <origin rpy="0 0 0" xyz="0.0064 0 0"/>
-      <!-- copied from proximal_actuating_hinge -->
-      <mass value="0.00362"/>
-      <inertia ixx="0.00000012043" ixy="0" ixz="0" iyy="0.00000053588" iyz="0" izz="0.00000065322"/>
-    </inertial>
-  </link>
-  <gazebo reference="l_finger_1_link_paraproximal_actuating_hinge">
-    <mu1>1.1</mu1>
-    <mu2>1.1</mu2>
-  </gazebo>
-  <!-- Link proximal actuating bar -->
-  <link name="l_finger_1_link_proximal_actuating_bar">
-    <visual>
-      <origin rpy="0 0 0" xyz="0.026789 0 0"/>
-      <geometry>
-        <box size="0.05398 .0075 .002"/>
-      </geometry>
-    </visual>
-    <collision>
-      <origin rpy="0 0 0" xyz="0.026789 0 0"/>
-      <geometry>
-        <box size="0.05398 .0075 .002"/>
-      </geometry>
-    </collision>
-    <inertial>
-      <origin rpy="0 0 0" xyz="0.02699 -0.00122 0"/>
-      <mass value="0.00659"/>
-      <inertia ixx="0.00000008348" ixy="-0.0000002179" ixz="0.00000000134" iyy="0.00000719076" iyz="0" izz="0.00000718272"/>
-    </inertial>
-  </link>
-  <gazebo reference="l_finger_1_link_proximal_actuating_bar">
-    <mu1>1.1</mu1>
-    <mu2>1.1</mu2>
-  </gazebo>
-  <!-- Link paraproximal bar -->
-  <link name="l_finger_1_link_paraproximal_bar">
-    <visual>
-      <origin rpy="0 0 0" xyz="0.02885 0 0"/>
-      <geometry>
-        <box size="0.05770 .0075 .002"/>
-      </geometry>
-    </visual>
-    <collision>
-      <origin rpy="0 0 0" xyz="0.02885 0 0"/>
-      <geometry>
-        <box size="0.05770 .0075 .002"/>
-      </geometry>
-    </collision>
-    <inertial>
-      <origin rpy="0 0 0" xyz="0.02858 -0.00129 0"/>
-      <mass value="0.00732"/>
-      <inertia ixx="0.00000009065" ixy="-0.00000027047" ixz="0.00000000142" iyy="0.00000878034" iyz="0" izz="0.00000877558"/>
-    </inertial>
-  </link>
-  <gazebo reference="l_finger_1_link_paraproximal_bar">
-    <mu1>1.1</mu1>
-    <mu2>1.1</mu2>
-  </gazebo>
-  <!-- Link median actuating hinge -->
-  <link name="l_finger_1_link_median_actuating_hinge">
-    <visual>
-      <origin rpy="0 0 0" xyz="0 0 0"/>
-      <geometry>
-        <box size=".02 .02 .002"/>
-      </geometry>
-    </visual>
-    <collision>
-      <origin rpy="0 0 0" xyz="0 0 0"/>
-      <geometry>
-        <box size=".02 .02 .002"/>
-      </geometry>
-    </collision>
-    <inertial>
-      <origin rpy="0 0 0" xyz="0.0092 0.00514 0"/>
-      <mass value="0.00359"/>
-      <inertia ixx="0.00000024735" ixy="0.00000023619" ixz="0" iyy="0.00000047681" iyz="0" izz="0.00000071813"/>
-    </inertial>
-  </link>
-  <gazebo reference="l_finger_1_link_median_actuating_hinge">
-    <mu1>1.1</mu1>
-    <mu2>1.1</mu2>
-  </gazebo>
-  <!-- Link median bar -->
-  <link name="l_finger_1_link_median_bar">
-    <visual>
-      <origin rpy="0 0 0" xyz="0.01905 0 0"/>
-      <geometry>
-        <box size="0.0381 .0075 .002"/>
-      </geometry>
-    </visual>
-    <collision>
-      <origin rpy="0 0 0" xyz="0.01905 0 0"/>
-      <geometry>
-        <box size="0.0381 .0075 .002"/>
-      </geometry>
-    </collision>
-    <inertial>
-      <origin rpy="0 0 0" xyz="0.01905 -0.00107 0"/>
-      <mass value="0.00538"/>
-      <inertia ixx="0.00000006639" ixy="-0.00000010996" ixz="0.00000000094" iyy="0.00000305318" iyz="0" izz="0.00000304657"/>
-    </inertial>
-  </link>
-  <gazebo reference="l_finger_1_link_median_bar">
-    <mu1>1.1</mu1>
-    <mu2>1.1</mu2>
-  </gazebo>
-  <!-- Link paramedian hinge -->
-  <link name="l_finger_1_link_paramedian_hinge">
-    <visual>
-      <origin rpy="0 0 0" xyz="0 0 0"/>
-      <geometry>
-        <box size=".02 .02 .002"/>
-      </geometry>
-    </visual>
-    <collision>
-      <origin rpy="0 0 0" xyz="0 0 0"/>
-      <geometry>
-        <box size=".02 .02 .002"/>
-      </geometry>
-    </collision>
-    <inertial>
-      <origin rpy="0 0 0" xyz="-0.01025 0.00046 0"/>
-      <mass value="0.00276"/>
-      <inertia ixx="0.00000004213" ixy="-0.00000001491" ixz="0" iyy="0.00000050258" iyz="0" izz="0.00000054007"/>
-    </inertial>
-  </link>
-  <gazebo reference="l_finger_1_link_paramedian_hinge">
-    <mu1>1.1</mu1>
-    <mu2>1.1</mu2>
-  </gazebo>
-  <!-- Link median bar underactuated -->
-  <link name="l_finger_1_link_median_bar_underactuated">
-    <visual>
-      <origin rpy="0 0 0" xyz="0.01905 0 0"/>
-      <geometry>
-        <box size="0.0381 .0075 .002"/>
-      </geometry>
-    </visual>
-    <collision>
-      <origin rpy="0 0 0" xyz="0.01905 0 0"/>
-      <geometry>
-        <box size="0.0381 .0075 .002"/>
-      </geometry>
-    </collision>
-    <inertial>
-      <origin rpy="0 0 0" xyz="0.01905 -0.00107 0"/>
-      <mass value="0.00538"/>
-      <inertia ixx="0.00000006639" ixy="-0.00000010996" ixz="-0.00000000094" iyy="0.00000305318" iyz="0" izz="0.00000304657"/>
-    </inertial>
-  </link>
-  <gazebo reference="l_finger_1_link_median_bar_underactuated">
-    <mu1>1.1</mu1>
-    <mu2>1.1</mu2>
-  </gazebo>
-  <!-- Link paradistal hinge -->
-  <link name="l_finger_1_link_paradistal_hinge">
-    <visual>
-      <origin rpy="0 0 0" xyz="0 0 0"/>
-      <geometry>
-        <box size=".02 .02 .002"/>
-      </geometry>
-    </visual>
-    <collision>
-      <origin rpy="0 0 0" xyz="0 0 0"/>
-      <geometry>
-        <box size=".02 0.02 .002"/>
-      </geometry>
-    </collision>
-    <inertial>
-      <origin rpy="0 0 0" xyz="0.00548 0 0"/>
-      <mass value="0.00158"/>
-      <inertia ixx="0.00000001907" ixy="0" ixz="0" iyy="0.00000010970" iyz="0" izz="0.00000012610"/>
-    </inertial>
-  </link>
-  <gazebo reference="l_finger_1_link_paradistal_hinge">
-    <mu1>1.1</mu1>
-    <mu2>1.1</mu2>
-  </gazebo>
-  <!-- End of link list -->
-  <!-- Joint list -->
-  <!-- Joint proximal actuating hinge -->
-  <joint name="l_finger_1_joint_proximal_actuating_hinge" type="revolute">
-    <parent link="l_finger_1_link_0"/>
-    <child link="l_finger_1_link_proximal_actuating_hinge"/>
-    <axis xyz="0 0 1"/>
-    <origin rpy="0 0 -2.0906" xyz="0 0 0.01"/>
-    <limit effort="100" lower="-3.1416" upper="3.1416" velocity="100"/>
-  </joint>
-  <gazebo reference="l_finger_1_joint_proximal_actuating_hinge">
-    <implicitSpringDamper>1</implicitSpringDamper>
-  </gazebo>
-  <!-- Joint paraproximal actuating hinge -->
-  <joint name="l_finger_1_joint_paraproximal_actuating_hinge" type="revolute">
-    <parent link="l_finger_1_link_0"/>
-    <child link="l_finger_1_link_paraproximal_actuating_hinge"/>
-    <axis xyz="0 0 1"/>
-    <origin rpy="0 0 -2.0906" xyz="0 0 -0.01"/>
-    <limit effort="100" lower="-3.1416" upper="3.1416" velocity="100"/>
-  </joint>
-  <gazebo reference="l_finger_1_joint_paraproximal_actuating_hinge">
-    <implicitSpringDamper>1</implicitSpringDamper>
-  </gazebo>
-  <!-- Joint proximal actuating bar -->
-  <joint name="l_finger_1_joint_proximal_actuating_bar" type="revolute">
-    <parent link="l_finger_1_link_proximal_actuating_hinge"/>
-    <child link="l_finger_1_link_proximal_actuating_bar"/>
-    <axis xyz="0 0 1"/>
-    <origin rpy="0 0 1.8616" xyz="0.02858 0 0"/>
-    <limit effort="100" lower="-3.1416" upper="3.1416" velocity="100"/>
-  </joint>
-  <gazebo reference="l_finger_1_joint_proximal_actuating_bar">
-    <implicitSpringDamper>1</implicitSpringDamper>
-  </gazebo>
-  <!-- Joint paraproximal bar -->
-  <joint name="l_finger_1_joint_paraproximal_bar" type="revolute">
-    <parent link="l_finger_1_link_paraproximal_actuating_hinge"/>
-    <child link="l_finger_1_link_paraproximal_bar"/>
-    <axis xyz="0 0 1"/>
-    <origin rpy="0 0 1.57" xyz="0.02286 0 0"/>
-    <limit effort="100" lower="-3.1416" upper="3.1416" velocity="100"/>
-  </joint>
-  <gazebo reference="l_finger_1_joint_paraproximal_bar">
-    <implicitSpringDamper>1</implicitSpringDamper>
-  </gazebo>
-  <!-- Joint median actuating hinge -->
-  <joint name="l_finger_1_joint_median_actuating_hinge" type="revolute">
-    <parent link="l_finger_1_link_1"/>
-    <child link="l_finger_1_link_median_actuating_hinge"/>
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
Commit message: Added velodyne frame

File: husky_description/urdf/dual_arm_husky.urdf.xacro (robot description, xacro)
@@ -345,4 +345,12 @@
     <origin rpy="0 0 0" xyz="0 0 0.225"/>
   </joint>
+  <!-- Velodyne Link -->
+  <link name="velodyne"/>
+  <!-- Attach Velodyne Link -->
+  <joint name="velodyne_joint" type="fixed">
+    <parent link="dual_arm_bulkhead_link"/>
+    <child link="velodyne"/>
+    <origin rpy="0 0 0" xyz="-0.24535 0 0.39296"/>
+  </joint>
   <link name="husky_ptu_pan_link">
     <inertial>
